File: termite.kicad_pcb (KiCad board)
At the start: 2 copper layers, 261.4 x 82.1 mm, 112 parts, among them J1 AudioJack4, J2 AudioJack4, SW1 SW_Push_45deg, SW10 SW_Push_45deg, SW11 SW_Push_45deg, SW12 SW_Push_45deg, SW13 SW_Push_45deg, SW14 SW_Push_45deg, SW15 SW_Push_45deg, SW16 SW_Push_45deg, SW17 SW_Push_45deg, SW18 SW_Push_45deg, SW19 SW_Push_45deg, SW2 SW_Push_45deg, SW20 SW_Push_45deg, SW21 SW_Push_45deg, SW22 SW_Push_45deg, SW23 SW_Push_45deg, SW24 SW_Push_45deg, SW25 SW_Push_45deg, SW26 SW_Push_45deg, SW27 SW_Push_45deg, SW28 SW_Push_45deg, SW29 SW_Push_45deg, SW3 SW_Push_45deg, SW30 SW_Push_45deg, SW31 SW_Push_45deg, SW32 SW_Push_45deg, SW33 SW_Push_45deg, SW34 SW_Push_45deg, SW4 SW_Push_45deg, SW5 SW_Push_45deg, SW6 SW_Push_45deg, SW7 SW_Push_45deg, SW8 SW_Push_45deg, SW9 SW_Push_45deg, U1 Pico, U2 Pico

Commit message: fix: bring jack connectors to the edge
Parts:
- moved R3 5.09 mm to (156.4, 84.6)
- moved R4 5.09 mm to (164.1, 86.8)
- moved J1 5.09 mm to (141.1, 89.7)
- moved J2 5.09 mm to (150.2, 89.7)
- moved R1 5.09 mm to (134.9, 84.6)
- moved R2 5.09 mm to (127.2, 91.8)
Routing:
- net GND_R: track 490.9 -> 500.7 mm
- net COL_R_2: track 212.7 -> 204.4 mm
- net VBUS_R: track 439.1 -> 446.7 mm
- net COL_R_4: track 163.6 -> 156.0 mm
- net COL_R_3: track 179.1 -> 171.7 mm
- net GND_L: track 510.3 -> 517.5 mm
- net COL_R_5: track 136.5 -> 129.9 mm
- net SCL_R_1: track 41.2 -> 45.8 mm
- net SCL_L_1: track 68.4 -> 63.9 mm
- net SDA_L_1: track 49.3 -> 44.8 mm
- net SDA_R_1: track 36.3 -> 40.2 mm, vias 0 -> 1
- net ROW_R_3: track 178.5 -> 182.0 mm
- net ROW_R_2: track 188.2 -> 191.6 mm
- net ROW_R_1: track 197.8 -> 201.0 mm
- net VBUS_L: track 452.2 -> 450.1 mm
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